File: trans & formador/trans & formador.kicad_sch (KiCad schematic)
At the start: 38 parts, among them J1 Saida Trafo, J2 Entrada Trafo, J3 Entrada AC, J4 Saida DC, J5 Led Curto, J6 Led ligado, J7 Potenciometro, J8 Led Curto

Commit message: Add files via upload
Parts:
- removed J2: Entrada Trafo, symbol Connector_Generic:Conn_01x02
- removed J3: Entrada AC, symbol Connector_Generic:Conn_01x02
- removed RP: 0,466, symbol Device:R
- removed RV1: Varistor, symbol Device:Varistor
- added C1: 10u, symbol Device:C_Polarized
- added DPR5, DPR6: 1N4002, Diode_THT:D_DO-41_SOD81_P10.16mm_Horizontal, symbol Diode:1N4002
- added R1: 10k, symbol Device:R
- added RP1, RP2: 0.233, symbol Device:R
- renumbered CF to CF1, CR to CR1, DZ to DZ1, QC to QC1, QZ to QZ1, RLC to RLC1, RLL to RLL1
Connections:
- net at CR1.2, DPR2.2 (A), DPR3.2 (A)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: now also C1.2, DPR5.2 (A), R1.2
- net at J4.1 (Pin_1), R11.2, R12.2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: now also C1.1, DPR5.1 (K), DPR6.2 (A), R1.1
- net at QA1.2 (C), QA2.2 (C), QA3.2 (C)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: now also RP2.2
- net at CR1.1, DPR1.1 (K), DPR4.1 (K)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: now also DPR6.1 (K), RP1.1
- new net: RP1.2, RP2.1
Other:
- moved on the sheet: J4

Commit message: Add files via upload
Parts:
- CR1: value C_Polarized -> 3300uF
- J8: value Led Curto -> Botao Curto
Changed lines of the file:
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@@
       (effects (font (size 1.27 1.27)) (justify left))
     )
-    (property "Value" "C_Polarized" (at 90.17 93.726 0)
+    (property "Value" "3300uF" (at 90.17 93.726 0)
       (effects (font (size 1.27 1.27)) (justify left))
     )
@@
       (effects (font (size 1.27 1.27)))
     )
-    (property "Value" "Led Curto" (at 127 123.19 0)
-      (effects (font (size 1.27 1.27)))
-    )
+    (property "Value" "Botao Curto" (at 127 123.19 0)
+      (effects (font (size 1.27 1.27)))
+    )
